Commit message: Updated to latest repo

File: tracebot_mockup_description/urdf/tracebot_mockup.urdf.xacro (robot description, xacro)
@@ -2,46 +2,17 @@
 <robot xmlns:xacro="http://wiki.ros.org/xacro" name="tracebot_mockup">
   <xacro:include filename="$(find tracebot_mockup_description)/urdf/tracebot_mockup_macro.urdf.xacro"/>
-  <xacro:include filename="$(find ur_description)/urdf/ur_macro.xacro"/>
   <!--Add parameters to robot base-->
   <xacro:tracebot_mockup
-    robot_mount_offset_x="$(arg robot_mount_offset_x)"
-    robot_mount_offset_y="$(arg robot_mount_offset_y)"
-    robot_mount_offset_z="$(arg robot_mount_offset_z)"
-    robot_mount_offset_theta="$(arg robot_mount_offset_theta)"
-    robot_mount_length="$(arg robot_mount_length)"
-    robot_mount_width="$(arg robot_mount_width)"
-    robot_mount_height="$(arg robot_mount_height)"
-    robot_base_tilt="$(arg robot_base_tilt)"
-    left_arm="$(arg left_arm)"
-    right_arm="$(arg right_arm)"/>
-  <!--Add parameters to robot arms-->
-  <xacro:ur_robot prefix="left_"
-    joint_limits_parameters_file="$(find ur_description)/config/$(arg left_arm)/joint_limits.yaml"
-    kinematics_parameters_file="$(find ur_description)/config/$(arg left_arm)/default_kinematics.yaml"
-    physical_parameters_file="$(find ur_description)/config/$(arg left_arm)/physical_parameters.yaml"
-    visual_parameters_file="$(find ur_description)/config/$(arg left_arm)/visual_parameters.yaml"
-    transmission_hw_interface="hardware_interface/VelocityJointInterface"
-    safety_limits="false"
-    safety_pos_margin="0.15"
-    safety_k_position="20"/>
-  <xacro:ur_robot prefix="right_"
-    joint_limits_parameters_file="$(find ur_description)/config/$(arg right_arm)/joint_limits.yaml"
-    kinematics_parameters_file="$(find ur_description)/config/$(arg right_arm)/default_kinematics.yaml"
-    physical_parameters_file="$(find ur_description)/config/$(arg right_arm)/physical_parameters.yaml"
-    visual_parameters_file="$(find ur_description)/config/$(arg right_arm)/visual_parameters.yaml"
-    transmission_hw_interface="hardware_interface/VelocityJointInterface"
-    safety_limits="false"
-    safety_pos_margin="0.15"
-    safety_k_position="20"/>
-  <!-- Link arms to base -->
-  <joint name="left_base_link_joint" type="fixed">
-    <origin xyz="0 0 0" rpy="0 0 1.5708"/>
-    <parent link="left_robot_mount"/>
-    <child link="left_base_link"/>
-  </joint>
-  <joint name="right_base_link_joint" type="fixed">
-    <origin xyz="0 0 0" rpy="0 0 -1.5708"/>
-    <parent link="right_robot_mount"/>
-    <child link="right_base_link"/>
-  </joint>
+    robot_name="$(arg robot_name)"
+    mount_base_width="$(arg mount_base_width)"
+    mount_base_length="$(arg mount_base_length)"
+    mount_base_height="$(arg mount_base_height)"
+    arm_mount_offset_x="$(arg arm_mount_offset_x)"
+    arm_mount_offset_y="$(arg arm_mount_offset_y)"
+    arm_mount_offset_z="$(arg arm_mount_offset_z)"
+    arm_mount_offset_theta="$(arg arm_mount_offset_theta)"
+    arm_base_tilt="$(arg arm_base_tilt)"
+    left_arm_model="$(arg left_arm_model)"
+    right_arm_model="$(arg right_arm_model)"
+  />
 </robot>

File: tracebot_mockup_description/urdf/tracebot_mockup_macro.urdf.xacro (robot description, xacro)
@@ -1,26 +1,27 @@
 <?xml version="1.0"?>
 <robot xmlns:xacro="http://wiki.ros.org/xacro">
-  <xacro:macro name="tracebot_mockup" params="robot_mount_offset_x
-                                              robot_mount_offset_y
-                                              robot_mount_offset_z
-                                              robot_mount_offset_theta
-                                              robot_mount_height
-                                              robot_mount_length
-                                              robot_mount_width
-                                              robot_base_tilt
-                                              left_arm
-                                              right_arm">
+  <xacro:macro name="tracebot_mockup" params="robot_name
+                                              mount_base_width
+                                              mount_base_length
+                                              mount_base_height
+                                              arm_mount_offset_x:=0
+                                              arm_mount_offset_y:=0
+                                              arm_mount_offset_z:=0
+                                              arm_mount_offset_theta:=0
+                                              arm_base_tilt:=0
+                                              left_arm_model
+                                              right_arm_model">
     <!-- Base -->
-    <link name="base_link"/>
-    <joint name="robot_mount_base_joint" type="fixed">
+    <link name="${robot_name}_base_link"/>
+    <joint name="${robot_name}_mount_base_joint" type="fixed">
       <origin xyz="0 0 0" rpy="0 0 0"/>
-      <parent link="base_link"/>
-      <child link="robot_mount_base"/>
+      <parent link="${robot_name}_base_link"/>
+      <child link="${robot_name}_arm_mount_base"/>
     </joint>
-    <link name="robot_mount_base">
+    <link name="${robot_name}_arm_mount_base">
       <visual>
-        <origin xyz="0 0 ${robot_mount_height/2}" rpy="0 0 0"/>
+        <origin xyz="0 0 ${mount_base_height/2}" rpy="0 0 0"/>
         <geometry>
-          <mesh filename="file:///home/benrjg/astech_wss/tracebot_mockup_ws/src/tracebot_mockup/tracebot_mockup_description/meshes/stand.stl" />
+          <mesh filename="package://tracebot_mockup_description/meshes/stand.stl" />
         </geometry>
         <material name="grey">
@@ -29,18 +30,48 @@
       </visual>
     </link>
+    <!-- Arm Setup -->
+    <xacro:include filename="$(find ur_description)/urdf/ur_macro.xacro"/>
     <!-- Left Arm Mount -->
-    <joint name="left_robot_mount_joint" type="fixed">
-      <origin xyz="${-robot_mount_offset_x} 0 ${robot_mount_height-robot_mount_offset_z}" rpy="0 ${-pi/2+robot_base_tilt} 0"/>
-      <parent link="robot_mount_base"/>
-      <child link="left_robot_mount"/>
+    <joint name="${robot_name}_left_arm_mount_joint" type="fixed">
+      <origin xyz="${-arm_mount_offset_x} 0 ${mount_base_height-arm_mount_offset_z}" rpy="0 ${-pi/2+arm_base_tilt} 0"/>
+      <parent link="${robot_name}_arm_mount_base"/>
+      <child link="${robot_name}_left_arm_mount"/>
     </joint>
-    <link name="left_robot_mount"/>
+    <link name="${robot_name}_left_arm_mount"/>
+    <joint name="${robot_name}_left_arm_base_link_joint" type="fixed">
+      <origin xyz="0 0 0" rpy="0 0 1.5708"/>
+      <parent link="${robot_name}_left_arm_mount"/>
+      <child link="${robot_name}_left_arm_base_link"/>
+    </joint>
+    <xacro:ur_robot prefix="${robot_name}_left_arm_"
+      joint_limits_parameters_file="$(find ur_description)/config/$(arg left_arm_model)/joint_limits.yaml"
+      kinematics_parameters_file="$(find ur_description)/config/$(arg left_arm_model)/default_kinematics.yaml"
+      physical_parameters_file="$(find ur_description)/config/$(arg left_arm_model)/physical_parameters.yaml"
+      visual_parameters_file="$(find ur_description)/config/$(arg left_arm_model)/visual_parameters.yaml"
+      transmission_hw_interface="hardware_interface/PositionJointInterface"
+      safety_limits="false"
+      safety_pos_margin="0.15"
+      safety_k_position="20"/>
     <!-- Right Arm Mount -->
-    <joint name="right_robot_mount_joint" type="fixed">
-      <origin xyz="${robot_mount_offset_x} 0 ${robot_mount_height-robot_mount_offset_z}" rpy="0 ${pi/2-robot_base_tilt} 0"/>
-      <parent link="robot_mount_base"/>
-      <child link="right_robot_mount"/>
+    <joint name="${robot_name}_right_arm_mount_joint" type="fixed">
+      <origin xyz="${arm_mount_offset_x} 0 ${mount_base_height-arm_mount_offset_z}" rpy="0 ${pi/2-arm_base_tilt} 0"/>
+      <parent link="${robot_name}_arm_mount_base"/>
+      <child link="${robot_name}_right_arm_mount"/>
     </joint>
-    <link name="right_robot_mount"/>
+    <link name="${robot_name}_right_arm_mount"/>
+    <joint name="${robot_name}_right_arm_base_link_joint" type="fixed">
+      <origin xyz="0 0 0" rpy="0 0 -1.5708"/>
+      <parent link="${robot_name}_right_arm_mount"/>
+      <child link="${robot_name}_right_arm_base_link"/>
+    </joint>
+    <xacro:ur_robot prefix="${robot_name}_right_arm_"
+      joint_limits_parameters_file="$(find ur_description)/config/$(arg right_arm_model)/joint_limits.yaml"
+      kinematics_parameters_file="$(find ur_description)/config/$(arg right_arm_model)/default_kinematics.yaml"
+      physical_parameters_file="$(find ur_description)/config/$(arg right_arm_model)/physical_parameters.yaml"
+      visual_parameters_file="$(find ur_description)/config/$(arg right_arm_model)/visual_parameters.yaml"
+      transmission_hw_interface="hardware_interface/PositionJointInterface"
+      safety_limits="false"
+      safety_pos_margin="0.15"
+      safety_k_position="20"/>
   </xacro:macro>
 </robot>

File: tracebot_mockup_gazebo/urdf/tracebot_mockup.urdf.xacro (robot description, xacro)
@@ -2,67 +2,40 @@
 <robot xmlns:xacro="http://wiki.ros.org/xacro" name="tracebot_mockup_gazebo">
   <xacro:include filename="$(find tracebot_mockup_gazebo)/urdf/tracebot_mockup_macro.urdf.xacro"/>
-  <xacro:include filename="$(find tracebot_mockup_gazebo)/urdf/ur_macro.xacro"/>
   <!--Robot base parameters-->
-  <xacro:arg name="robot_mount_offset_x" default="0.1293"/>
-  <xacro:arg name="robot_mount_offset_y" default="0.0"/>
-  <xacro:arg name="robot_mount_offset_z" default="0.0707"/>
-  <xacro:arg name="robot_mount_offset_theta" default="0.0"/>
-  <xacro:arg name="robot_mount_length" default="0.55"/>
-  <xacro:arg name="robot_mount_width" default="0.55"/>
-  <xacro:arg name="robot_mount_height" default="1.2664"/>
-  <xacro:arg name="robot_base_tilt" default="0.785398"/>
-  <xacro:arg name="left_arm" default="ur5e"/>
-  <xacro:arg name="right_arm" default="ur5e"/>
+  <xacro:arg name="robot_name" default="tracebot"/>
+  <xacro:arg name="mount_base_width" default="0.55"/>
+  <xacro:arg name="mount_base_length" default="0.55"/>
+  <xacro:arg name="mount_base_height" default="1.27"/>
+  <xacro:arg name="arm_mount_offset_x" default="0.1293"/>
+  <xacro:arg name="arm_mount_offset_y" default="0.0"/>
+  <xacro:arg name="arm_mount_offset_z" default="0.0707"/>
+  <xacro:arg name="arm_mount_offset_theta" default="0.0"/>
+  <xacro:arg name="arm_base_tilt" default="0.785398"/>
+  <xacro:arg name="left_arm_model" default="ur5e"/>
+  <xacro:arg name="right_arm_model" default="ur5e"/>
   <!--Robot arm parameters-->
   <xacro:arg name="transmission_hw_interface" default="hardware_interface/PositionJointInterface"/>
   <!--Add parameters to robot base-->
   <xacro:tracebot_mockup_gazebo
-    robot_mount_offset_x="$(arg robot_mount_offset_x)"
-    robot_mount_offset_y="$(arg robot_mount_offset_y)"
-    robot_mount_offset_z="$(arg robot_mount_offset_z)"
-    robot_mount_offset_theta="$(arg robot_mount_offset_theta)"
-    robot_mount_length="$(arg robot_mount_length)"
-    robot_mount_width="$(arg robot_mount_width)"
-    robot_mount_height="$(arg robot_mount_height)"
-    robot_base_tilt="$(arg robot_base_tilt)"
-    left_arm="$(arg left_arm)"
-    right_arm="$(arg right_arm)"/>
-  <!--Add parameters to robot arms-->
-  <xacro:ur_robot_gazebo prefix="left_"
-    joint_limits_parameters_file="$(find ur_description)/config/$(arg left_arm)/joint_limits.yaml"
-    kinematics_parameters_file="$(find ur_description)/config/$(arg left_arm)/default_kinematics.yaml"
-    physical_parameters_file="$(find ur_description)/config/$(arg left_arm)/physical_parameters.yaml"
-    visual_parameters_file="$(find ur_description)/config/$(arg left_arm)/visual_parameters.yaml"
-    transmission_hw_interface="$(arg transmission_hw_interface)"
-    safety_limits="false"
-    safety_pos_margin="0.15"
-    safety_k_position="20"/>
-  <xacro:ur_robot_gazebo prefix="right_"
-    joint_limits_parameters_file="$(find ur_description)/config/$(arg right_arm)/joint_limits.yaml"
-    kinematics_parameters_file="$(find ur_description)/config/$(arg right_arm)/default_kinematics.yaml"
-    physical_parameters_file="$(find ur_description)/config/$(arg right_arm)/physical_parameters.yaml"
-    visual_parameters_file="$(find ur_description)/config/$(arg right_arm)/visual_parameters.yaml"
-    transmission_hw_interface="$(arg transmission_hw_interface)"
-    safety_limits="false"
-    safety_pos_margin="0.15"
-    safety_k_position="20"/>
-  <!--Link arms to base-->
-  <joint name="left_base_link_joint" type="fixed">
-    <origin xyz="0 0 0" rpy="0 0 1.5708"/>
-    <parent link="left_robot_mount"/>
-    <child link="left_base_link"/>
-  </joint>
-  <joint name="right_base_link_joint" type="fixed">
-    <origin xyz="0 0 0" rpy="0 0 -1.5708"/>
-    <parent link="right_robot_mount"/>
-    <child link="right_base_link"/>
-  </joint>
+    robot_name="$(arg robot_name)"
+    mount_base_width="$(arg mount_base_width)"
+    mount_base_length="$(arg mount_base_length)"
+    mount_base_height="$(arg mount_base_height)"
+    arm_mount_offset_x="$(arg arm_mount_offset_x)"
+    arm_mount_offset_y="$(arg arm_mount_offset_y)"
+    arm_mount_offset_z="$(arg arm_mount_offset_z)"
+    arm_mount_offset_theta="$(arg arm_mount_offset_theta)"
+    arm_base_tilt="$(arg arm_base_tilt)"
+    left_arm_model="$(arg left_arm_model)"
+    right_arm_model="$(arg right_arm_model)"
+  />
   <!--Link base to world-->
   <link name="world"/>
   <joint name="world_joint" type="fixed">
     <parent link="world"/>
-    <child link="base_link"/>
+    <child link="$(arg robot_name)_base_link"/>
     <origin xyz="0 0 0" rpy="0 0 0"/>
   </joint>
+  <!-- Gazebo ROS Plugins -->
   <gazebo>
     <plugin name="ros_control" filename="libgazebo_ros_control.so">

File: tracebot_mockup_gazebo/urdf/tracebot_mockup_macro.urdf.xacro (robot description, xacro)
@@ -1,31 +1,77 @@
 <?xml version="1.0"?>
 <robot xmlns:xacro="http://wiki.ros.org/xacro">
-  <xacro:macro name="tracebot_mockup_gazebo" params="
-    robot_mount_offset_x
-    robot_mount_offset_y
-    robot_mount_offset_z
-    robot_mount_offset_theta
-    robot_mount_height
-    robot_mount_length
-    robot_mount_width
-    robot_base_tilt
-    left_arm
-    right_arm">
+  <xacro:macro name="tracebot_mockup_gazebo" params="robot_name
+                                                     mount_base_width
+                                                     mount_base_length
+                                                     mount_base_height
+                                                     arm_mount_offset_x:=0
+                                                     arm_mount_offset_y:=0
+                                                     arm_mount_offset_z:=0
+                                                     arm_mount_offset_theta:=0
+                                                     arm_base_tilt:=0
+                                                     left_arm_model
+                                                     right_arm_model">
     <xacro:include filename="$(find tracebot_mockup_description)/urdf/tracebot_mockup_macro.urdf.xacro"/>
     <!--Pass arguments to tracebot_mockup-->
     <xacro:tracebot_mockup
-      robot_mount_offset_x="${robot_mount_offset_x}"
-      robot_mount_offset_y="${robot_mount_offset_y}"
-      robot_mount_offset_z="${robot_mount_offset_z}"
-      robot_mount_offset_theta="${robot_mount_offset_theta}"
-      robot_mount_height="${robot_mount_height}"
-      robot_mount_length="${robot_mount_length}"
-      robot_mount_width="${robot_mount_width}"
-      robot_base_tilt="${robot_base_tilt}"
-      left_arm="${left_arm}"
-      right_arm="${right_arm}"
+      robot_name="$(arg robot_name)"
+      mount_base_width="$(arg mount_base_width)"
+      mount_base_length="$(arg mount_base_length)"
+      mount_base_height="$(arg mount_base_height)"
+      arm_mount_offset_x="$(arg arm_mount_offset_x)"
+      arm_mount_offset_y="$(arg arm_mount_offset_y)"
+      arm_mount_offset_z="$(arg arm_mount_offset_z)"
+      arm_mount_offset_theta="$(arg arm_mount_offset_theta)"
+      arm_base_tilt="$(arg arm_base_tilt)"
+      left_arm_model="$(arg left_arm_model)"
+      right_arm_model="$(arg right_arm_model)"
     />
-    <!--Add collision to base-->
-    <gazebo reference="robot_mount_base">
+    <!-- Configure self collision properties per link -->
+    <!-- Base Collision -->
+    <gazebo reference="${robot_name}_mount_base">
+      <selfCollide>true</selfCollide>
+    </gazebo>
+    <!-- Left Arm Collision -->
+    <gazebo reference="${robot_name}_left_arm_shoulder_link">
+      <selfCollide>true</selfCollide>
+    </gazebo>
+    <gazebo reference="${robot_name}_left_arm_upper_arm_link">
+      <selfCollide>true</selfCollide>
+    </gazebo>
+    <gazebo reference="${robot_name}_left_arm_forearm_link">
+      <selfCollide>true</selfCollide>
+    </gazebo>
+    <gazebo reference="${robot_name}_left_arm_wrist_1_link">
+      <selfCollide>true</selfCollide>
+    </gazebo>
+    <gazebo reference="${robot_name}_left_arm_wrist_3_link">
+      <selfCollide>true</selfCollide>
+    </gazebo>
+    <gazebo reference="${robot_name}_left_arm_wrist_2_link">
+      <selfCollide>true</selfCollide>
+    </gazebo>
+    <gazebo reference="${robot_name}_left_arm_ee_link">
+      <selfCollide>true</selfCollide>
+    </gazebo>
+    <!-- Right Arm Collision -->
+    <gazebo reference="${robot_name}_right_arm_shoulder_link">
+      <selfCollide>true</selfCollide>
+    </gazebo>
+    <gazebo reference="${robot_name}_right_arm_upper_arm_link">
+      <selfCollide>true</selfCollide>
+    </gazebo>
+    <gazebo reference="${robot_name}_right_arm_forearm_link">
+      <selfCollide>true</selfCollide>
+    </gazebo>
+    <gazebo reference="${robot_name}_right_arm_wrist_1_link">
+      <selfCollide>true</selfCollide>
+    </gazebo>
+    <gazebo reference="${robot_name}_right_arm_wrist_3_link">
+      <selfCollide>true</selfCollide>
+    </gazebo>
+    <gazebo reference="${robot_name}_right_arm_wrist_2_link">
+      <selfCollide>true</selfCollide>
+    </gazebo>
+    <gazebo reference="${robot_name}_right_arm_ee_link">
       <selfCollide>true</selfCollide>
     </gazebo>
